File: serial-usb-adapter.kicad_pcb (KiCad board)
At the start: 2 copper layers, 38 x 26 mm, 30 parts, among them J1 USB_B_Micro, J2 UART Header, J3 USB Power, U1 LPC47M192, U2 FT231XS, Y1 SG5032CAN 14.318MHz

Commit message: Break out SMI output pin & set thermal spoke width to 0.3 mm for power pads
Parts:
- added R7: 1k, Resistor_SMD:R_0603_1608Metric, B.Cu at (108.3, 128.5)
- added ~{SMI}: , SMD1,27-2,54, F.Cu at (94.7, 132.2)
- moved C9 1.10 mm to (109.8, 128.5), turned to 90 degrees
Connections:
- JP1 pad 12: (no net) -> VSS
- JP1 pad 15: VCC -> (no net)
- U1 pad 50: (no net) -> SMI
Routing:
- net SMI: track 0.00 -> 16.9 mm, vias 0 -> 1
- net VCC: track 72.3 -> 64.1 mm
- net VBUS: vias 2 -> 1
